File: design/design.kicad_sch (KiCad schematic)
At the start: 1 part, among them U1 ESP32-DevKitC

Commit message: started schematic
Parts:
- added C1, C2: 100u, symbol Device:C_Small
- added D1: LED, symbol Device:LED
- added J1: Conn_01x08_Socket, Connector_JST:JST_XH_B8B-XH-A_1x08_P2.50mm_Vertical, symbol Connector:Conn_01x08_Socket
- added J2: Conn_01x06_Socket, Connector_JST:JST_XH_B6B-XH-A_1x06_P2.50mm_Vertical, symbol Connector:Conn_01x06_Socket
- added Q1, Q2: NPN, symbol Simulation_SPICE:NPN
- added R_1: 250?, symbol Device:R_Small_US
- added R_2, R_4, R_6: 1k, symbol Device:R_Small_US
- added R_3: 100, symbol Device:R_Small_US
- added R_5: 100k, symbol Device:R_Small_US
- added R_7: 60k, symbol Device:R_Small_US
- added U2, U3: TL072, symbol Amplifier_Operational:TL072
Connections:
- net GND: now also C1.2, D1.1 (K), R_2.2, R_5.2, R_6.1
- net O_AMP_REG: now reaches U1.10 (DAC_2/ADC2_CH9/GPIO26)
- net O_AMP_REG: now also U2.3 (+)
- net O_KEYPAD_ROW_0: now reaches U1.11 (ADC2_CH7/GPIO27)
- net O_KEYPAD_ROW_0: now also J1.1 (Pin_1)
- net O_KEYPAD_ROW_1: now reaches U1.12 (MTMS/GPIO14/ADC2_CH6)
- net O_KEYPAD_ROW_1: now also J1.2 (Pin_2)
- net O_KEYPAD_ROW_2: now reaches U1.13 (MTDI/GPIO12/ADC2_CH5)
- net O_KEYPAD_ROW_2: now also J1.3 (Pin_3)
- net O_KEYPAD_ROW_3: now reaches U1.15 (MTCK/GPIO13/ADC2_CH4)
- net O_KEYPAD_ROW_3: now also J1.4 (Pin_4)
- net O_OFFSET_POSITIVE: now reaches U1.16 (SD_DATA2/GPIO9)
- net O_OFFSET_NEGATIVE: now reaches U1.17 (SD_DATA3/GPIO10)
- net O_STATUS_LED: now reaches U1.18 (CMD)
- net O_STATUS_LED: now also R_1.1
- net VCC: now reaches U1.19 (5V)
- net VCC: now also R_4.1
- net I_KEYPAD_COL_3: now reaches U1.23 (MTDO/GPIO15/ADC2_CH3)
- net I_KEYPAD_COL_3: now also J1.8 (Pin_8)
- net I_KEYPAD_COL_0: now reaches U1.27 (GPIO16)
- net I_KEYPAD_COL_0: now also J1.5 (Pin_5)
- net O_LCD_DATA_PIN_3: now reaches U1.29 (GPIO5)
- net O_LCD_DATA_PIN_3: now also J2.4 (Pin_4)
- net O_LCD_DATA_PIN_1: now reaches U1.30 (GPIO18)
- net O_LCD_DATA_PIN_1: now also J2.2 (Pin_2)
- net O_LCD_DATA_PIN_0: now reaches U1.31 (GPIO19)
- net O_LCD_DATA_PIN_0: now also J2.1 (Pin_1)
- net O_LCD_DATA_PIN_2: now reaches U1.33 (GPIO21)
- net O_LCD_DATA_PIN_2: now also J2.3 (Pin_3)
- net O_LCD_ENABLE: now reaches U1.36 (GPIO22)
- net O_LCD_ENABLE: now also J2.6 (Pin_6)
- net O_LCD_REG_SELECT: now reaches U1.37 (GPIO23)
- net O_LCD_REG_SELECT: now also J2.5 (Pin_5)
- net I_KEYPAD_COL_2: now reaches U1.7 (32K_XP/GPIO32/ADC1_CH4)
- net I_KEYPAD_COL_2: now also J1.7 (Pin_7)
- net I_KEYPAD_COL_1: now reaches U1.8 (32K_XN/GPIO33/ADC1_CH5)
- net I_KEYPAD_COL_1: now also J1.6 (Pin_6)
- net O_SIGNAL: now reaches U1.9 (DAC_1/ADC2_CH8/GPIO25)
- net O_SIGNAL: now also Q2.2 (B)
- new net: R_6.2, R_7.1, U3.2 (-)
- new net: Q1.3 (E), R_2.1, U2.2 (-)
- new net: R_3.1, U2.1
- new net: Q1.2 (B), R_3.2
- new net: C1.1, Q1.1 (C), Q2.3 (E)
- new net: C2.2, R_5.1, U3.3 (+)
- new net: C2.1, Q2.1 (C), R_4.2
- new net: R_7.2, U3.1
- new net: D1.2 (A), R_1.2
Other:
- note added: "Green"
- note added: "Keypad JST Connector"
- note added: "LCD JST Connector"

Commit message: initial schematic done
Parts:
- added C3: 100u, symbol Device:C_Small
- added C4, C6: 33n, symbol Device:C_Small
- added C5, C7: 68n, symbol Device:C_Small
- added R_10: 2k, symbol Device:R_Small_US
- added R_11, R_15, R_9: 1k, symbol Device:R_Small_US
- added R_12, R_13, R_14: 100k, symbol Device:R_Small_US
- added R_16: 11k, symbol Device:R_Small_US
- added R_17, R_18, R_19, R_20: 8.2k, symbol Device:R_Small_US
- added R_21, R_22, R_25, R_26, R_27: 10k, symbol Device:R_Small_US
- added R_23, R_24: 40k, symbol Device:R_Small_US
- added R_8: 300k, symbol Device:R_Small_US
- added U4, U5, U6, U7, U8, U9: TL072, symbol Amplifier_Operational:TL072
Connections:
- net GND: now also C4.2, C6.2, R_11.1, R_16.2, R_24.2, R_9.1, U5.3 (+), U9.3 (+); no longer R_2.2
- net O_AMP_REG: now also R_10.1; no longer U2.3 (+)
- net O_OFFSET_NEGATIVE: now also R_17.2
- net O_OFFSET_POSITIVE: now also R_19.2
- net O_SIGNAL: now also C3.1; no longer Q2.2 (B)
- net VCC: now also R_15.1
- net AC_SIGNAL: now reaches R_7.2, U3.1
- net AC_SIGNAL: now also R_26.2
- net I_REG_SENSE: now reaches U1.3 (SENSOR_VP/GPIO36/ADC1_CH0)
- new net: C7.1, R_19.1, R_20.2
- new net: C7.2, R_21.2, U7.1, U7.2 (-)
- new net: R_25.1, R_26.1, R_27.2, U9.2 (-)
- new net: R_12.1, R_13.2, R_14.1, U5.2 (-)
- new net: C3.2, R_8.1
- new net: R_22.1, R_24.1, U8.3 (+)
- new net: C5.2, R_22.2, U6.1, U6.2 (-)
- new net: C6.1, R_20.1, U7.3 (+)
- new net: R_21.1, R_23.2, U8.2 (-)
- new net: C5.1, R_17.1, R_18.2
- new net: C4.1, R_18.1, U6.3 (+)
- new net: Q2.2 (B), U4.1, U4.2 (-)
- new net: R_8.2, R_9.2, U4.3 (+)
- new net: R_14.2, R_15.2, R_16.1
- new net: R_10.2, R_11.2, R_12.2
- new net DC_OFFSET: R_23.1, R_25.2, U8.1
- new net OUTPUT: R_27.1, U9.1
- new net REG: R_13.1, U2.3 (+), U5.1
- new net VEE: R_2.2
Other:
- note added: "DAC 0 to 3.3V lerp to range -11 to -12V"
- note added: "Final adder"
- note added: "MCU"
- note added: "Main DAC signal output to AC signal precise amplifier"
- note added: "Note: OpAmps have to be powered by a greater voltage than VCC"
- note added: "PWM signals through Sallen-Key lowpass into differetial amplifier"
- note added: "Same note"
- moved on the sheet: C1, C2, D1, J1, J2, Q1, Q2, R_1, R_2, R_3, R_4, R_5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
