File: design/design.kicad_sch (KiCad schematic)
At the start: 22 parts, among them J1 Conn_01x08_Socket, Q1 NPN, Q2 NPN, U1 ESP32-DevKitC, U2 TL072, U4 TL072, U5 TL072

Commit message: cleanup
Parts:
- removed R_10: 1.75k, symbol Device:R_Small_US
- removed R_11: 1k, symbol Device:R_Small_US
- added R_7: 3k, symbol Device:R_Small_US
- added R_8: 1k, symbol Device:R_Small_US
- R_6: renamed from R_8; value 600k -> 6k
- R_9: value 1k -> 10
Connections:
- net +3V3: no longer R1.1, R_4.1
- net GND: now also R_8.2
- net I_REG_SENSE: no longer C2.2, R_5.1
- net O_AMP_REG: now also U2.3 (+)
- net VCC: now also R1.1, R_4.1
- net at U5.3 (+): now also C2.2, R_5.1
- removed net REG: U2.3 (+), U5.1, U5.2 (-)
- new net: R_7.1, R_8.1, U5.2 (-)
- new net: R_7.2, U5.1
Other:
- note removed: "DAC 0 to 3.3V lerp to 0-1.2V"

Commit message: cleanup the schematic
Parts:
- removed R_2, R_4, R_8: 1k, symbol Device:R_Small_US
- removed R_3: 100, symbol Device:R_Small_US
- removed R_5: 100k, symbol Device:R_Small_US
- removed R_6: 6k, symbol Device:R_Small_US
- removed R_7: 3k, symbol Device:R_Small_US
- removed R_9: 10, symbol Device:R_Small_US
- removed U5: TL072, symbol Amplifier_Operational:TL072
- added R10, R3, R5, R8: 1k, symbol Device:R_Small_US
- added R4: 2k, symbol Device:R_Small_US
- added R6: 100k, symbol Device:R_Small_US
- added R7: 3k, symbol Device:R_Small_US
- added R9: 100, symbol Device:R_Small_US
- added U3: TL072, Package_DFN_QFN:Texas_DSQ0010A_WSON-10-1EP_2x2mm_P0.4mm_EP0.9x1.5mm, symbol Amplifier_Operational:TL072
- C1, C2, C3: footprint (none) -> Package_SO:SOIC-8_3.9x4.9mm_P1.27mm
- Q1, Q2: footprint (none) -> Package_DFN_QFN:Nordic_AQFN-94-1EP_7x7mm_P0.4mm
- R1: value 1k -> 6k; footprint Package_DIP:DIP-8_W7.62mm -> (none)
- R2: value 2k -> 10; footprint Package_DIP:DIP-8_W7.62mm -> (none)
- U2, U4: footprint (none) -> Package_DFN_QFN:Texas_DSQ0010A_WSON-10-1EP_2x2mm_P0.4mm_EP0.9x1.5mm
Connections:
- net GND: now also C3.1, R2.1, R10.1, R4.1, R6.1, R8.1; no longer C1.2, R2.2
- net I_REG_SENSE: now also R7.1, U3.1
- net O_AMP_REG: now also U4.3 (+); no longer U2.3 (+)
- net O_SIGNAL: now also R1.1
- net VCC: now also R3.2, R5.2; no longer R1.1
- net at Q1.3 (E): now also C3.2, Q2.1 (C); no longer U2.2 (-)
- net at U2.1: now also C1.1, U2.2 (-)
- net at Q1.2 (B): now also C1.2, R3.1, R4.2
- net at C2.2: now also R6.2, U3.3 (+)
- net at C2.1: now also Q1.1 (C), R5.1; no longer Q2.1 (C)
- new net: Q2.2 (B), R9.1
- new net: R9.2, U4.1
- new net: R7.2, R8.2, U3.2 (-)
- new net: R1.2, R2.2, U2.3 (+)
- new net: Q2.3 (E), R10.2, U4.2 (-)
Other:
- moved on the sheet: D1, J1, R_1, U1
