File: design/_autosave-design.kicad_sch (KiCad schematic)
At the start: 22 parts, among them J1 Conn_01x08_Socket, Q1 NPN, Q2 NPN, U1 ESP32-DevKitC, U2 TL072, U4 TL072, U5 TL072

Commit message: improve precise amplifier circuit
Parts:
- removed R_10: 1.75k, symbol Device:R_Small_US
- removed R_11: 1k, symbol Device:R_Small_US
- removed U5: TL072, symbol Amplifier_Operational:TL072
- R_6: renamed from R_8; value 600k -> 6k
- R_9: value 1k -> 10
Connections:
- net REG is gone; now on net O_AMP_REG: U2.3 (+)
- net +3V3: no longer R1.1, R_4.1
- net VCC: now also R1.1, R_4.1
Other:
- note removed: "DAC 0 to 3.3V lerp to 0-1.2V"

Commit message: add a new amplifying stage at the output
Parts:
- added R_7: 3k, symbol Device:R_Small_US
- added R_8: 1k, symbol Device:R_Small_US
- added U5: TL072, symbol Amplifier_Operational:TL072
Connections:
- net GND: now also R_8.2
- net I_REG_SENSE: no longer C2.2, R_5.1
- new net: R_7.1, R_8.1, U5.2 (-)
- new net: C2.2, R_5.1, U5.3 (+)
- new net: R_7.2, U5.1
